Commit message: Fix init height, base_height_target, and optimize collision bodies
- boying_config: pos_z 0.35→0.16m, base_height_target 0.30→0.14m
  (actual standing height ~0.13m, previous values caused 0.22m freefall on reset)
- boying_config: add Method B PD params as comments (k=26, d=0.64)
- URDF: extend base collision box to 0.430×0.185×0.136m
- URDF: thigh cylinder length 0.04→0.07m, origin_y moved inward 0.02m
- URDF: thigh box size 0.03×0.03×0.23m, origin adjusted
- URDF: calf cylinder length 0.18→0.22m

Co-Authored-By: Claude Sonnet 4.6 <noreply@anthropic.com>

File: legged_gym/resources/robots/boying_description/urdf/boying_description_withouthm.urdf (robot description, URDF)
Before this commit: robot boying, 19 links, 18 joints
Links:
- link FL_thigh: geometry collision box size=0.03 0.03 0.23; collision cylinder length=0.0700 radius=0.044
- link FR_thigh: geometry collision box size=0.03 0.03 0.23; collision cylinder length=0.0700 radius=0.044
- link RL_thigh: geometry collision box size=0.03 0.03 0.23; collision cylinder length=0.0700 radius=0.044
- link RR_thigh: geometry collision box size=0.03 0.03 0.23; collision cylinder length=0.0700 radius=0.044
- link base: geometry collision box size=0.430 0.185 0.136; visual mesh filename=../meshes/base.STL

Commit message: Adjust collision bodies and revert init height params
- boying_config: pos_z reverted to 0.40m, base_height_target to 0.32
- URDF: thigh cylinder moved outward 1cm along y-axis (FL/RL: 0.100→0.110, FR/RR: -0.100→-0.110)
- URDF: base collision box y-axis reduced 0.5cm (0.185→0.180m)

Co-Authored-By: Claude Sonnet 4.6 <noreply@anthropic.com>

File: legged_gym/resources/robots/boying_description/urdf/boying_description_withouthm.urdf (robot description, URDF)
Before this commit: robot boying, 19 links, 18 joints
Links:
- link base: geometry collision box size=0.430 0.180 0.136; visual mesh filename=../meshes/base.STL
